Commit message: 이제그만

File: simulation/urdf/camera.urdf.xacro (robot description, xacro)
@@ -4,5 +4,5 @@
         <gazebo reference="camera_link">
             <sensor name="camera" type="camera">
-                <pose>0 0 0 0 3.141592653589793 3.141592653589793</pose>
+                <pose>0 0 0 0 0 0</pose>
                 <always_on>true</always_on>
                 <visualize>true</visualize>

File: simulation/urdf/my_rover.urdf.xacro (robot description, xacro)
@@ -133,5 +133,5 @@
     <parent link="base_link"/>
     <child link="camera_link"/>
-    <origin xyz="0.495 0 0.155" rpy="0 0 0"/>
+    <origin xyz="0.495 0 0.155" rpy="0 3.14159 3.14159"/>
   </joint>
   <gazebo>
